File: Hardware/Venturi_MainPCB/Venturi_MainPCB.kicad_sch (KiCad schematic)
At the start: 75 parts, among them J1 Battery, J2 ESC_PWM, J3 ESC_P, J4 ESC_N, J5 M1, J6 M1, J7 Sensor-PCB, Q1 BSS138, Q2 DMP3013SFV, U1 TSOP38238, U2 ESP32-P4-WIFI6, U3 MIC29152WU, U4 DRV8212P, U5 DRV8212P, U6 ICM-20948

Commit message: Updated PCB-Design for 20MHz SPI speed
Parts:
- removed C17, C18, C24, C7: 100n, Capacitor_SMD:C_0805_2012Metric_Pad1.18x1.45mm_HandSolder, symbol Device:C
- removed C6, C8: 100uF, Capacitor_Tantalum_SMD:CP_EIA-7343-15_Kemet-W_HandSolder, symbol Device:C_Polarized
- removed D2, D3: LED, LED_SMD:LED_0805_2012Metric_Pad1.15x1.40mm_HandSolder, symbol Device:LED
- removed JP1: POWER_EN, TestPoint:TestPoint_2Pads_Pitch2.54mm_Drill0.8mm, symbol Jumper:Jumper_2_Open
- removed JP2: ESP_EN, TestPoint:TestPoint_2Pads_Pitch2.54mm_Drill0.8mm, symbol Jumper:Jumper_2_Open
- removed R13: 10k, Resistor_SMD:R_0805_2012Metric_Pad1.20x1.40mm_HandSolder, symbol Device:R
- removed R2, R3: 330R, Resistor_SMD:R_0805_2012Metric_Pad1.20x1.40mm_HandSolder, symbol Device:R
- removed U6: ICM-20948, Sensor_Motion:InvenSense_QFN-24_3x3mm_P0.4mm, symbol Sensor_Motion:ICM-20948
- added C15, C16, C5: 220uF, Capacitor_SMD:CP_Elec_6.3x9.9, symbol Device:C_Polarized
- added H10, H11, H12, H9: (no value), MountingHole:MountingHole_3.2mm_M3_DIN965, symbol Mechanical:MountingHole
- added R10, R11: 22R, Resistor_SMD:R_0805_2012Metric_Pad1.20x1.40mm_HandSolder, symbol Device:R
- added SW1: POWER_EN, Button_Switch_SMD:SW_SPST_Omron_B3FS-100xP, symbol Switch:SW_Omron_B3FS
- added U6: ICM-42670-P, Package_LGA:LGA-14_3x2.5mm_P0.5mm_LayoutBorder3x4y, symbol Sensor_Motion:ICM-42670-P
- C2, C3, C4: value 100uF -> 220uF; footprint Capacitor_Tantalum_SMD:CP_EIA-7343-15_Kemet-W_HandSolder -> Capacitor_SMD:CP_Elec_6.3x9.9
- R12: value 3k3 -> 22R
- renumbered C12 to C10, C13 to C11, C14 to C12, C15 to C13, C16 to C14, C19 to C17, C20 to C18, C22 to C19, C21 to C20, C23 to C21, C5 to C6, C9 to C7, C10 to C8, C11 to C9, D4 to D2, D5 to D3, D6 to D4, D7 to D5, D8 to D6, D9 to D7, R14 to R13, R15 to R14, R16 to R15, R11 to R2, R4 to R3, R5 to R4, R6 to R5, R7 to R6, R8 to R7, R9 to R8, R10 to R9
Connections:
- net +3V3: now also J7.5 (Pin_5), J7.6 (Pin_6), R15.1, U6.5 (VDDIO), U6.8 (VDD); no longer J7.10 (Pin_10), J7.11 (Pin_11), R12.1
- net +BATT: now also C15.1, C16.1, C5.1
- net CLK: now also J7.12 (Pin_12), R11.2; no longer J7.4 (Pin_4), U2.8 (GPIO3)
- net CS: now also J7.14 (Pin_14), R10.2; no longer J7.2 (Pin_2), U2.7 (GPIO2)
- net GND: now also J7.11 (Pin_11), J7.13 (Pin_13), J7.4 (Pin_4), C15.2, C16.2, C5.2, U6.6 (GND), U6.7 (FSYNC); no longer J7.12 (Pin_12), J7.3 (Pin_3), J7.5 (Pin_5), R15.2
- net IMU_INT: now also R15.2, U6.4 (INT1/INT); no longer R15.1
- net MOSI: now also J7.10 (Pin_10), R12.2; no longer J7.6 (Pin_6), U2.9 (GPIO4)
- net SK6812: now also U2.18 (GPIO27); no longer U2.15 (GPIO22)
- net VCC: now also J7.2 (Pin_2), J7.3 (Pin_3); no longer J7.13 (Pin_13), J7.14 (Pin_14)
- net at Q1.3 (D), Q2.4 (G), R4.2: now also SW1.2
- net at R1.1: now also U2.20 (GPIO29); no longer U2.16 (GPIO23)
- net at R3.1: now also SW1.1
- net IMU_MISO: now reaches U2.13 (GPIO20)
- net IMU_MISO: now also U6.1 (AP_SDO/AP_AD0)
- net IMU_MOSI: now reaches U2.14 (GPIO21)
- net IMU_MOSI: now also U6.14 (AP_SDI)
- net IMU_SCL: no longer names the net of U2.12 (GPIO8)
- net IMU_SCL: no longer R12.2
- net IMU_SDA: no longer names the net of U2.11 (GPIO7)
- net IMU_SDA: no longer R2.2
- new net: R11.1, U2.8 (GPIO3)
- new net: R10.1, U2.7 (GPIO2)
- new net: R12.1, U2.9 (GPIO4)
- new net IMU_CLK: U2.15 (GPIO22), U6.13 (AP_SCL/AP_SCLK)
- new net IMU_CS: R2.2, U2.16 (GPIO23), U6.12 (AP_CS)
Other:
- moved on the sheet: C19, C21, J2, J3, J4, J7, R15, R2
