File: Hardware/Venturi_MainPCB/Venturi_MainPCB.kicad_sch (KiCad schematic)
At the start: 72 parts, among them J1 Battery, J2 ESC_PWM, J3 ESC_P, J4 ESC_N, J5 M1, J6 M1, J7 Sensor-PCB, Q1 BSS138, Q2 DMP3013SFV, SW1 POWER_EN, U1 TSOP38238, U2 ESP32-P4-WIFI6, U3 MIC29152WU, U4 DRV8212P, U5 DRV8212P, U6 ICM-42670-P

Commit message: Added Typst Documentation
Parts:
- removed R10, R11, R12: 22R, Resistor_SMD:R_0805_2012Metric_Pad1.20x1.40mm_HandSolder, symbol Device:R
- removed U2: ESP32-P4-WIFI6, RF_Module:ESP32-P4-WIFI6, symbol RF_Module:ESP32-P4-WIFI6
- added C1, C6, C9: 100n, Capacitor_SMD:C_0805_2012Metric_Pad1.18x1.45mm_HandSolder, symbol Device:C
- added C16: 10u, Capacitor_SMD:C_0603_1608Metric_Pad1.08x0.95mm_HandSolder, symbol Device:C
- added C21: 2.2n, Capacitor_SMD:C_0603_1608Metric_Pad1.08x0.95mm_HandSolder, symbol Device:C
- added C22: 100n, Capacitor_SMD:C_0603_1608Metric_Pad1.08x0.95mm_HandSolder, symbol Device:C
- added C26, C27, C29: 22u, Capacitor_SMD:C_0603_1608Metric_Pad1.08x0.95mm_HandSolder, symbol Device:C
- added D1: BAT54C, Package_TO_SOT_SMD:SOT-23, symbol Diode:BAT54C
- added D9: LED, LED_SMD:LED_0805_2012Metric_Pad1.15x1.40mm_HandSolder, symbol Device:LED
- added F1: 500mA, Fuse:Fuse_0805_2012Metric_Pad1.15x1.40mm_HandSolder, symbol Device:Fuse
- added IC1: TS3USB221DRCR, Package_SON:SON50P300X300X100-11N-D, symbol UniversalProgrammer:TS3USB221DRCR
- added J5: Micro_SD_Card, Connector_Card:microSD_HC_Wuerth_693072010801, symbol Connector:Micro_SD_Card
- added J6: USB_C_Receptacle_USB2.0_14P, Connector_USB:USB_C_Receptacle_G-Switch_GT-USB-7010ASV, symbol Connector:USB_C_Receptacle_USB2.0_14P
- added L1: 3u3, Inductor_SMD:L_Vishay_IHLP-1616, symbol Device:L
- added Q3: BSS138, Package_TO_SOT_SMD:SOT-23, symbol Transistor_FET:BSS138
- added R14, R15, R16, R17, R18, R19, R20, R9: 10k, Resistor_SMD:R_0805_2012Metric_Pad1.20x1.40mm_HandSolder, symbol Device:R
- added R23, R24: 5k1, Resistor_SMD:R_0805_2012Metric_Pad1.20x1.40mm_HandSolder, symbol Device:R
- added R25, R26: 10k, Resistor_SMD:R_0603_1608Metric_Pad0.98x0.95mm_HandSolder, symbol Device:R
- added R27, R28, R6, R7, R8: 22R, Resistor_SMD:R_0805_2012Metric_Pad1.20x1.40mm_HandSolder, symbol Device:R
- added R29: 47k, Resistor_SMD:R_0603_1608Metric_Pad0.98x0.95mm_HandSolder, symbol Device:R
- added R30: 15k, Resistor_SMD:R_0603_1608Metric_Pad0.98x0.95mm_HandSolder, symbol Device:R
- added R32: 68k, Resistor_SMD:R_0603_1608Metric_Pad0.98x0.95mm_HandSolder, symbol Device:R
- added R33: 1k, Resistor_SMD:R_0603_1608Metric_Pad0.98x0.95mm_HandSolder, symbol Device:R
- added R34: 22k, Resistor_SMD:R_0603_1608Metric_Pad0.98x0.95mm_HandSolder, symbol Device:R
- added R35: 330R, Resistor_SMD:R_0603_1608Metric_Pad0.98x0.95mm_HandSolder, symbol Device:R
- added SW2: ESP_EN, Button_Switch_SMD:SW_SPST_Omron_B3FS-100xP, symbol Switch:SW_Omron_B3FS
- added SW3: ESP_BOOT, Button_Switch_SMD:SW_SPST_Omron_B3FS-100xP, symbol Switch:SW_Omron_B3FS
- added U2: ESP32-S31-WROOM-3, RF_Module:ESP32-S31-WROOM-3, symbol RF_Module:ESP32-S31-WROOM-3
- added U4: SLogic16U3, Custom:SLogic16U3, symbol Custom:SLogic16U3
- added U5: USBLC6-2P6, Package_TO_SOT_SMD:SOT-666, symbol Power_Protection:USBLC6-2P6
- added U8: AP64500SP-13, Package_SO:SO-8EP_DIO, symbol Regulator_Linear:AP64500SP-13
- J8: renamed from J6; value M1 -> M2
- U1: footprint OptoDevice:Vishay_MINICAST-3Pin -> OptoDevice:Vishay_CAST-3Pin
- renumbered C7 to C10, C8 to C11, C9 to C12, C12 to C13, C13 to C14, C10 to C15, C11 to C17, C15 to C18, C16 to C19, C1 to C2, C14 to C20, C17 to C23, C19 to C24, C18 to C25, C20 to C28, C2 to C3, C21 to C30, C3 to C4, C4 to C5, C5 to C7, C6 to C8, D1 to D2, D2 to D3, D3 to D4, D4 to D5, D5 to D6, D6 to D7, D7 to D8, J5 to J7, J7 to J9, R3 to R1, R6 to R10, R7 to R11, R8 to R12, R9 to R13, R1 to R2, R13 to R21, R14 to R22, R2 to R3, R15 to R31, U4 to U6, U5 to U7, U6 to U9
Connections:
- net +3V3: now also C26.2, C27.2, C29.2, C6.1, D9.2 (A), J5.4 (VDD), L1.2, R14.1, R15.1, R16.1, R17.1, R18.1, R19.1, R20.1, R32.1, R9.1, U2.3 (3V3), U2.4 (3V3)
- net +BATT: now also C16.2, U8.2 (VIN), U8.3 (EN)
- net CLK: now also R7.2, U4.7 (Pin_7)
- net CS: now also R6.2, U4.8 (Pin_8)
- net GND: now also C1.1, C16.1, C21.2, C26.1, C27.1, C29.1, C6.2, C9.2, IC1.11 (EP), IC1.5 (GND), IC1.9 (S), J5.6 (VSS), J5.SH (SHIELD), J6.A1 (GND), J6.A12 (GND), J6.B1 (GND), J6.B12 (GND), J6.SH (SHIELD), Q3.2 (S), R23.2, R24.2, R26.2, R29.2, R34.2, R35.2, SW2.1, SW3.2, U2.1 (GND), U2.2 (GND), U2.26 (GND), U2.33 (NC), U2.34 (NC), U2.35 (NC), U2.36 (NC), U2.37 (NC), U2.38 (NC), U2.39 (NC), U2.47 (GND), U2.48 (GND), U2.72 (GND), U2.73 (GND), U2.74 (GND), U2.75 (GND), U2.76 (GND), U2.77 (GND), U2.78 (GND), U2.79 (GND), U2.80 (GND), U2.81 (GND), U2.82 (GND), U2.83 (GND), U2.84 (GND), U2.85 (GND), U2.86 (GND), U2.87 (GND), U2.88 (GND), U2.89 (GND), U2.90 (GND), U2.91 (NC), U2.92 (GND), U2.93 (GND), U2.94 (GND), U2.95 (GND), U2.96 (GND), U2.97 (GND), U2.98 (GND), U2.99 (GND), U4.GND, U5.2 (GND), U8.7 (GND), U8.EPAD (GND)
- net IMU_CLK: now also U2.19 (IO13), U4.3 (Pin_3)
- net IMU_CS: now also U2.20 (IO14), U4.4 (Pin_4)
- net IMU_INT: now also U2.55 (IO45)
- net IMU_MISO: now also U2.17 (IO11), U4.1 (Pin_1)
- net IMU_MOSI: now also U2.18 (IO12), U4.2 (Pin_2)
- net IR_SENSOR: now also U2.15 (IO9)
- net MA_ENC_A: now also U2.53 (IO43), U4.13 (Pin_13)
- net MA_ENC_B: now also U2.52 (IO42), U4.14 (Pin_14)
- net MA_OUT_1: now also U2.49 (IO38), U4.9 (Pin_9)
- net MA_OUT_2: now also U2.46 (IO37), U4.10 (Pin_10)
- net MB_ENC_A: now also U2.51 (IO40), U4.15 (Pin_15)
- net MB_ENC_B: now also U2.50 (IO39), U4.16 (Pin_16)
- net MB_OUT_1: now also U2.45 (IO36), U4.11 (Pin_11)
- net MB_OUT_2: now also U2.44 (IO35), U4.12 (Pin_12)
- net MISO: now also U2.24 (IO18), U4.5 (Pin_5)
- net MOSI: now also R8.2, U4.6 (Pin_6)
- net POWER_EN: now also D1.1, U2.54 (IO44); no longer Q1.1 (G), R5.1
- net SK6812: now also U2.16 (IO10)
- net VBAT: now also U2.56 (IO46)
- net at R2.1: now also U2.25 (IO19)
- net at J2.1 (Pin_1): now also U2.14 (IO8)
- net USB_EN: now reaches J1.2 (Pin_2), Q2.1 (S), Q2.2 (S), Q2.3 (S), R4.1
- net USB_EN: now also Q3.1 (G), R26.1
- new net: D1.3, Q1.1 (G), R5.1
- new net: C22.1, U8.1 (BST)
- new net: R29.1, U8.4 (RT/CLK)
- new net: R33.2, R34.1, U8.5 (FB)
- new net: R30.1, U8.6 (COMP)
- new net: C22.2, L1.1, U8.8 (SW)
- new net: F1.1, J6.A4 (VBUS), J6.A9 (VBUS), J6.B4 (VBUS), J6.B9 (VBUS)
- new net: J6.A5 (CC1), R24.1
- new net: J6.A6 (D+), J6.B6 (D+), U5.3 (I/O2)
- new net: J6.A7 (D-), J6.B7 (D-), U5.1 (I/O1)
- new net: J6.B5 (CC2), R23.1
- new net: C21.1, R30.2
- new net: C9.1, R15.2, SW3.1, U2.71 (IO61)
- new net: R6.1, U2.21 (IO15)
- new net: IC1.2 (1D-), R28.1
- new net: D9.1 (K), R35.1
- new net: IC1.1 (1D+), R27.1
- new net: IC1.6 (~{OE}), Q3.3 (D), R25.2
- new net: R32.2, R33.1
- new net: C1.2, R9.2, SW2.2, U2.5 (EN)
- new net: R7.1, U2.22 (IO16)
- new net: R8.1, U2.23 (IO17)
- new net: R14.2, U2.70 (IO60)
- new net D+: IC1.8 (D+), U5.4 (I/O2)
- new net D-: IC1.7 (D-), U5.6 (I/O1)
- new net ESP_D+: R27.2, U2.40 (USB_DP)
- new net ESP_D-: R28.2, U2.41 (USB_DM)
- new net SD_CLK: J5.5 (CLK), U2.29 (SD_D2)
- new net SD_CMD: J5.3 (CMD), R18.2, U2.30 (SD_D3)
- new net SD_D0: J5.7 (DAT0), R19.2, U2.28 (SD_D1)
- new net SD_D1: J5.8 (DAT1), R20.2, U2.27 (SD_D0)
- new net SD_D2: J5.1 (DAT2), R16.2, U2.32 (SD_CMD)
- new net SD_D3: J5.2 (DAT3/CD), R17.2, U2.31 (SD_CLK)
- new net VBUS: D1.2, F1.2, IC1.10 (VCC), R25.1, U5.5 (VBUS)
- no-connect marks 0 -> 3
Other:
- moved on the sheet: C10, C11, C12, C13, C14, C15, C17, C18, C19, C2, C20, C23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

Commit message: Updated PCB fonts and part name and value placing
Parts:
- X5: renamed from J6; value USB_C_Receptacle_USB2.0_14P -> USB-C
- renumbered U9 to B1, C24 to C1, C2 to C13, C19 to C14, C14 to C15, C15 to C16, C20 to C18, C23 to C19, C30 to C2, C25 to C20, C28 to C21, C16 to C23, C26 to C24, C27 to C25, C29 to C26, C21 to C27, C6 to C28, C1 to C29, C9 to C30, C7 to C6, C18 to C7, C13 to C8, C8 to C9, U6 to D1, IC1 to D2, U7 to D3, D3 to D4, D4 to D5, D5 to D6, D6 to D7, D7 to D8, D8 to D9, H8 to H10, H10 to H11, D2 to H13, H9 to H8, H11 to H9, U3 to N1, U8 to N2, U2 to N3, U4 to P1, R4 to R1, R23 to R10, R24 to R11, R26 to R12, R21 to R13, R22 to R14, R12 to R15, R13 to R16, R16 to R17, R17 to R18, R18 to R19, R10 to R2, R19 to R20, R20 to R21, R32 to R22, R29 to R23, R30 to R24, R33 to R25, R35 to R26, R34 to R27, R9 to R28, R14 to R29, R31 to R3, R15 to R30, R3 to R31, R6 to R32, R7 to R33, R8 to R34, R2 to R35, R1 to R4, R11 to R6, R27 to R7, R28 to R8, R25 to R9, Q2 to V1, Q1 to V2, U5 to V3, D1 to V4, Q3 to V5, U1 to V6, D9 to V7, J3 to X1, J1 to X2, J4 to X3, J7 to X4, J8 to X6, J9 to X7, J5 to X8, J2 to X9
