File: Hardware/Venturi_SensorPCB/Venturi_SensorPCB.kicad_pcb (KiCad board)
At the start: 4 copper layers, 162.6 x 31.2 mm, 60 parts, among them IC1 ADS7961SDBT, J1 Sensor-PCB, Q1 BSS138, Q2 BSS138, U1 QRE1113GR, U10 QRE1113GR, U11 QRE1113GR, U12 QRE1113GR, U13 QRE1113GR, U14 QRE1113GR, U15 QRE1113GR, U16 QRE1113GR, U2 QRE1113GR, U3 QRE1113GR, U4 QRE1113GR, U5 QRE1113GR, U6 QRE1113GR, U7 QRE1113GR, U8 QRE1113GR, U9 QRE1113GR

Commit message: Updated PCB-Design for 20MHz SPI speed
Parts:
- added R14: 3k3, Resistor_SMD:R_0805_2012Metric_Pad1.20x1.40mm_HandSolder, F.Cu at (152.3, 64.5)
- renumbered R14 to R15, R15 to R16, R16 to R17, R17 to R18, R18 to R19, R19 to R20, R20 to R21, R21 to R22, R22 to R23, R23 to R24, R24 to R25, R25 to R26, R26 to R27, R27 to R28, R28 to R29
Connections:
- IC1 pad 34: MISO -> Net-(IC1-SDO)
Routing:
- net Net-(IC1-SDO): track 0.00 -> 3.98 mm, vias 0 -> 1
- net GND: track 65.5 -> 63.9 mm, vias 216 -> 213
- net MOSI: track 11.5 -> 12.6 mm
- net CLK: track 11.9 -> 13.0 mm
- net CS: track 12.7 -> 13.8 mm
- net Net-(IC1-GPIO0): track 91.8 -> 92.8 mm
- net MISO: track 9.44 -> 8.91 mm, vias 0 -> 1
