File: Hardware/Venturi_SensorPCB/Venturi_SensorPCB.kicad_pcb (KiCad board)
At the start: 4 copper layers, 162.6 x 31.2 mm, 61 parts, among them IC1 ADS7961SDBT, J1 Sensor-PCB, Q1 BSS138, Q2 BSS138, U1 QRE1113GR, U10 QRE1113GR, U11 QRE1113GR, U12 QRE1113GR, U13 QRE1113GR, U14 QRE1113GR, U15 QRE1113GR, U16 QRE1113GR, U2 QRE1113GR, U3 QRE1113GR, U4 QRE1113GR, U5 QRE1113GR, U6 QRE1113GR, U7 QRE1113GR, U8 QRE1113GR, U9 QRE1113GR

Commit message: Updated PCB fonts and part name and value placing
Parts:
- R14: value 3k3 -> 22R
- renumbered D1 to H5, D2 to H6, IC1 to U1, U1 to V1, U10 to V10, U11 to V11, U12 to V12, Q1 to V13, Q2 to V14, U13 to V15, U14 to V16, U15 to V17, U16 to V18, U2 to V2, U3 to V3, U4 to V4, U5 to V5, U6 to V6, U7 to V7, U8 to V8, U9 to V9, J1 to X1
