File: Hardware/Venturi_SensorPCB/Venturi_SensorPCB.kicad_sch (KiCad schematic)
At the start: 61 parts, among them IC1 ADS7961SDBT, J1 Sensor-PCB, Q1 BSS138, Q2 BSS138, U1 QRE1113GR, U10 QRE1113GR, U11 QRE1113GR, U12 QRE1113GR, U13 QRE1113GR, U14 QRE1113GR, U15 QRE1113GR, U16 QRE1113GR, U2 QRE1113GR, U3 QRE1113GR, U4 QRE1113GR, U5 QRE1113GR, U6 QRE1113GR, U7 QRE1113GR, U8 QRE1113GR, U9 QRE1113GR

Commit message: Updated PCB fonts and part name and value placing
Parts:
- renumbered D1 to H5, D2 to H6, IC1 to U1, U1 to V1, U10 to V10, U11 to V11, U12 to V12, Q1 to V13, Q2 to V14, U13 to V15, U14 to V16, U15 to V17, U16 to V18, U2 to V2, U3 to V3, U4 to V4, U5 to V5, U6 to V6, U7 to V7, U8 to V8, U9 to V9, J1 to X1
Changed lines of the file:
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@@
 		(dnp no)
 		(fields_autoplaced yes)
-		(property "Reference" "U11"
+		(property "Reference" "V11"
 			(at 240.03 162.56 0)
 			(show_name no)
@@
 			(project "Venturi_SensorPCB"
 				(path "/179da9ab-1703-43d9-a037-538492c203c2"
-					(reference "U11")
+					(reference "V11")
 					(unit 1)
 				)
@@
 		(dnp no)
 		(fields_autoplaced yes)
-		(property "Reference" "U5"
+		(property "Reference" "V5"
 			(at 125.73 162.56 0)
 			(show_name no)
@@
 			(project "Venturi_SensorPCB"
 				(path "/179da9ab-1703-43d9-a037-538492c203c2"
-					(reference "U5")
+					(reference "V5")
 					(unit 1)
 				)
@@
 		(dnp no)
 		(fields_autoplaced yes)
-		(property "Reference" "U2"
+		(property "Reference" "V2"
 			(at 49.53 187.96 0)
 			(show_name no)
@@
 			(project "Venturi_SensorPCB"
 				(path "/179da9ab-1703-43d9-a037-538492c203c2"
-					(reference "U2")
+					(reference "V2")
 					(unit 1)
 				)
@@
 		(dnp no)
 		(fields_autoplaced yes)
-		(property "Reference" "U1"
+		(property "Reference" "V1"
 			(at 49.53 162.56 0)
 			(show_name no)
@@
 			(project "Venturi_SensorPCB"
 				(path "/179da9ab-1703-43d9-a037-538492c203c2"
-					(reference "U1")
+					(reference "V1")
 					(unit 1)
 				)
@@
 		(dnp no)
 		(fields_autoplaced yes)
-		(property "Reference" "U13"
+		(property "Reference" "V15"
 			(at 278.13 162.56 0)
 			(show_name no)
@@
 			(project "Venturi_SensorPCB"
 				(path "/179da9ab-1703-43d9-a037-538492c203c2"
-					(reference "U13")
+					(reference "V15")
 					(unit 1)
 				)
@@
 		(dnp no)
 		(fields_autoplaced yes)
-		(property "Reference" "U14"
+		(property "Reference" "V16"
 			(at 278.13 187.96 0)
 			(show_name no)
@@
 			(project "Venturi_SensorPCB"
 				(path "/179da9ab-1703-43d9-a037-538492c203c2"
-					(reference "U14")
+					(reference "V16")
 					(unit 1)
 				)
@@
 		(dnp no)
 		(fields_autoplaced yes)
-		(property "Reference" "U16"
+		(property "Reference" "V18"
 			(at 316.23 187.96 0)
 			(show_name no)
@@
 			(project "Venturi_SensorPCB"
 				(path "/179da9ab-1703-43d9-a037-538492c203c2"
-					(reference "U16")
+					(reference "V18")
 					(unit 1)
 				)
@@
 		(dnp no)
 		(fields_autoplaced yes)
-		(property "Reference" "U12"
+		(property "Reference" "V12"
 			(at 240.03 187.96 0)
 			(show_name no)
@@
 			(project "Venturi_SensorPCB"
 				(path "/179da9ab-1703-43d9-a037-538492c203c2"
-					(reference "U12")
+					(reference "V12")
 					(unit 1)
 				)
@@
 		(dnp no)
 		(fields_autoplaced yes)
-		(property "Reference" "U4"
+		(property "Reference" "V4"
 			(at 87.63 187.96 0)
 			(show_name no)
@@
 			(project "Venturi_SensorPCB"
 				(path "/179da9ab-1703-43d9-a037-538492c203c2"
-					(reference "U4")
+					(reference "V4")
 					(unit 1)
 				)
@@
 		(dnp no)
 		(fields_autoplaced yes)
-		(property "Reference" "Q2"
+		(property "Reference" "V14"
 			(at 281.94 55.8799 0)
 			(show_name no)
@@
 			(project "Venturi_SensorPCB"
 				(path "/179da9ab-1703-43d9-a037-538492c203c2"
-					(reference "Q2")
+					(reference "V14")
 					(unit 1)
 				)
@@
 		(dnp no)
 		(fields_autoplaced yes)
-		(property "Reference" "Q1"
+		(property "Reference" "V13"
 			(at 250.19 55.8799 0)
 			(show_name no)
@@
 			(project "Venturi_SensorPCB"
 				(path "/179da9ab-1703-43d9-a037-538492c203c2"
-					(reference "Q1")
+					(reference "V13")
 					(unit 1)
 				)
@@
 		(dnp no)
 		(fields_autoplaced yes)
-		(property "Reference" "D2"
+		(property "Reference" "H6"
 			(at 281.94 32.0674 90)
 			(show_name no)
@@
 			(project "Venturi_SensorPCB"
 				(path "/179da9ab-1703-43d9-a037-538492c203c2"
-					(reference "D2")
+					(reference "H6")
 					(unit 1)
 				)
@@
 		(dnp no)
 		(fields_autoplaced yes)
-		(property "Reference" "U9"
+		(property "Reference" "V9"
 			(at 201.93 162.56 0)
 			(show_name no)
@@
 			(project "Venturi_SensorPCB"
 				(path "/179da9ab-1703-43d9-a037-538492c203c2"
-					(reference "U9")
+					(reference "V9")
 					(unit 1)
 				)
@@
 		(in_pos_files yes)
 		(dnp no)
-		(property "Reference" "J1"
+		(property "Reference" "X1"
 			(at 76.2 49.5301 0)
 			(show_name no)
@@
 			(project "Venturi_SensorPCB"
 				(path "/179da9ab-1703-43d9-a037-538492c203c2"
-					(reference "J1")
+					(reference "X1")
 					(unit 1)
 				)
@@
 		(dnp no)
 		(fields_autoplaced yes)
-		(property "Reference" "U6"
+		(property "Reference" "V6"
 			(at 125.73 187.96 0)
 			(show_name no)
@@
 			(project "Venturi_SensorPCB"
 				(path "/179da9ab-1703-43d9-a037-538492c203c2"
-					(reference "U6")
+					(reference "V6")
 					(unit 1)
 				)
@@
 		(dnp no)
 		(fields_autoplaced yes)
-		(property "Reference" "U15"
+		(property "Reference" "V17"
 			(at 316.23 162.56 0)
 			(show_name no)
@@
 			(project "Venturi_SensorPCB"
 				(path "/179da9ab-1703-43d9-a037-538492c203c2"
-					(reference "U15")
+					(reference "V17")
 					(unit 1)
 				)
@@
 		(dnp no)
 		(fields_autoplaced yes)
-		(property "Reference" "IC1"
+		(property "Reference" "U1"
 			(at 163.83 30.48 0)
 			(show_name no)
@@
 			(project "Venturi_SensorPCB"
 				(path "/179da9ab-1703-43d9-a037-538492c203c2"
-					(reference "IC1")
+					(reference "U1")
 					(unit 1)
 				)
@@
 		(dnp no)
 		(fields_autoplaced yes)
-		(property "Reference" "U8"
+		(property "Reference" "V8"
 			(at 163.83 187.96 0)
 			(show_name no)
@@
 			(project "Venturi_SensorPCB"
 				(path "/179da9ab-1703-43d9-a037-538492c203c2"
-					(reference "U8")
+					(reference "V8")
 					(unit 1)
 				)
@@
 		(dnp no)
 		(fields_autoplaced yes)
-		(property "Reference" "D1"
+		(property "Reference" "H5"
 			(at 250.19 32.0674 90)
 			(show_name no)
@@
 			(project "Venturi_SensorPCB"
 				(path "/179da9ab-1703-43d9-a037-538492c203c2"
-					(reference "D1")
+					(reference "H5")
 					(unit 1)
 				)
@@
 		(dnp no)
 		(fields_autoplaced yes)
-		(property "Reference" "U3"
+		(property "Reference" "V3"
 			(at 87.63 162.56 0)
 			(show_name no)
@@
 			(project "Venturi_SensorPCB"
 				(path "/179da9ab-1703-43d9-a037-538492c203c2"
-					(reference "U3")
+					(reference "V3")
 					(unit 1)
 				)
@@
 		(dnp no)
 		(fields_autoplaced yes)
-		(property "Reference" "U10"
+		(property "Reference" "V10"
 			(at 201.93 187.96 0)
 			(show_name no)
@@
 			(project "Venturi_SensorPCB"
 				(path "/179da9ab-1703-43d9-a037-538492c203c2"
-					(reference "U10")
+					(reference "V10")
 					(unit 1)
 				)
@@
 		(dnp no)
 		(fields_autoplaced yes)
-		(property "Reference" "U7"
+		(property "Reference" "V7"
 			(at 163.83 162.56 0)
 			(show_name no)
@@
 			(project "Venturi_SensorPCB"
 				(path "/179da9ab-1703-43d9-a037-538492c203c2"
-					(reference "U7")
+					(reference "V7")
 					(unit 1)
 				)
